File: Pi5-plate/Pi5-plate.kicad_pcb (KiCad board)
At the start: 2 copper layers, 241.6 x 90.5 mm, 7 parts

Commit message: Pi5 Keyboard revision 1.
Parts:
- removed H5, H6: MountingHole_Pad, MountingHole:MountingHole_2.2mm_M2
- added D1: MountingHole, custom:Diode-slot, F.Cu at (50.8, 72.2)
- added D10: MountingHole, custom:Diode-slot, F.Cu at (234.2, 72.2)
- added D11: MountingHole, custom:Diode-slot, F.Cu at (48.1, 91.0)
- added D12: MountingHole, custom:Diode-slot, F.Cu at (66.9, 93.7)
- added D13: MountingHole, custom:Diode-slot, F.Cu at (85.7, 96.3)
- added D14: MountingHole, custom:Diode-slot, F.Cu at (104.6, 98.9)
- added D15: MountingHole, custom:Diode-slot, F.Cu at (123.4, 101.6)
- added D16: MountingHole, custom:Diode-slot, F.Cu at (161.6, 101.6)
- added D17: MountingHole, custom:Diode-slot, F.Cu at (180.4, 98.9)
- added D18: MountingHole, custom:Diode-slot, F.Cu at (199.3, 96.3)
- added D19: MountingHole, custom:Diode-slot, F.Cu at (218.1, 93.7)
- added D2: MountingHole, custom:Diode-slot, F.Cu at (69.6, 74.8)
- added D20: MountingHole, custom:Diode-slot, F.Cu at (236.9, 91.0)
- added D21: MountingHole, custom:Diode-slot, F.Cu at (45.5, 109.8)
- added D22: MountingHole, custom:Diode-slot, F.Cu at (64.3, 112.5)
- added D23: MountingHole, custom:Diode-slot, F.Cu at (83.1, 115.1)
- added D24: MountingHole, custom:Diode-slot, F.Cu at (101.9, 117.8)
- added D25: MountingHole, custom:Diode-slot, F.Cu at (120.7, 120.4)
- added D26: MountingHole, custom:Diode-slot, F.Cu at (164.3, 120.4)
- added D27: MountingHole, custom:Diode-slot, F.Cu at (183.1, 117.8)
- added D28: MountingHole, custom:Diode-slot, F.Cu at (201.9, 115.1)
- added D29: MountingHole, custom:Diode-slot, F.Cu at (220.7, 112.5)
- added D3: MountingHole, custom:Diode-slot, F.Cu at (88.4, 77.5)
- added D30: MountingHole, custom:Diode-slot, F.Cu at (239.5, 109.8)
- added D31: MountingHole, custom:Diode-slot, F.Cu at (42.8, 128.6)
- added D33: MountingHole, custom:Diode-slot, F.Cu at (80.4, 133.9)
- added D34: MountingHole, custom:Diode-slot, F.Cu at (99.3, 136.6)
- added D35: MountingHole, custom:Diode-slot, F.Cu at (118.1, 139.2)
- added D36: MountingHole, custom:Diode-slot, F.Cu at (166.9, 139.2)
- added D37: MountingHole, custom:Diode-slot, F.Cu at (185.7, 136.6)
- added D38: MountingHole, custom:Diode-slot, F.Cu at (204.6, 133.9)
- added D4: MountingHole, custom:Diode-slot, F.Cu at (107.2, 80.1)
- added D40: MountingHole, custom:Diode-slot, F.Cu at (242.2, 128.6)
- added D5: MountingHole, custom:Diode-slot, F.Cu at (126.0, 82.8)
- added D6: MountingHole, custom:Diode-slot, F.Cu at (159.0, 82.8)
- added D7: MountingHole, custom:Diode-slot, F.Cu at (177.8, 80.1)
- added D8: MountingHole, custom:Diode-slot, F.Cu at (196.6, 77.5)
- added D9: MountingHole, custom:Diode-slot, F.Cu at (215.4, 74.8)
