File: Pi5-plate/Pi5-plate.kicad_sch (KiCad schematic)
At the start: 6 parts

Commit message: Pi5 Keyboard revision 1.
Parts:
- removed H5, H6: MountingHole_Pad, MountingHole:MountingHole_2.2mm_M2, symbol Mechanical:MountingHole
- added D1, D10, D11, D12, D13, D14, D15, D16, D17, D18, D19, D2, D20, D21, D22, D23, D24, D25, D26, D27, D28, D29, D3, D30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: MountingHole, custom:Diode-slot, symbol Mechanical:MountingHole
