File: Pi5-pcb/Pi5-pcb.kicad_pcb (KiCad board)
At the start: 2 copper layers, 241.6 x 90.5 mm, 87 parts, among them J1 QWIIC, J2 DISPLAY, SW1 SW_Push, SW10 SW_Push, SW100 RESET, SW11 SW_Push, SW12 SW_Push, SW13 SW_Push, SW14 SW_Push, SW15 SW_Push, SW16 SW_Push, SW17 SW_Push, SW18 SW_Push, SW19 SW_Push, SW2 SW_Push, SW20 SW_Push, SW21 SW_Push, SW22 SW_Push, SW23 SW_Push, SW24 SW_Push, SW25 SW_Push, SW26 SW_Push, SW27 SW_Push, SW28 SW_Push, SW29 SW_Push, SW3 SW_Push, SW30 SW_Push, SW31 SW_Push, SW33 SW_Push, SW34 SW_Push, SW35 SW_Push, SW36 SW_Push, SW37 SW_Push, SW38 SW_Push, SW4 SW_Push, SW40 SW_Push, SW5 SW_Push, SW6 SW_Push, SW7 SW_Push, SW8 SW_Push, SW9 SW_Push, U1 Pico

Commit message: Pi5 Keyboard revision 1.
Parts:
- removed H6: MountingHole_Pad, MountingHole:MountingHole_2.2mm_M2
- H5: footprint MountingHole:MountingHole_2.2mm_M2 -> custom:PiPico-Mounting
- U1: footprint MCU_RaspberryPi_and_Boards:RPi_Pico_SMD_TH -> custom:PiPico
- moved H5 35.3 mm to (142.5, 99.0)
- moved SW100 1.30 mm to (147.3, 139.8)
Routing:
- net SCL0: track 27.5 -> 31.7 mm
- net SDA0: track 26.0 -> 29.0 mm
- net +3V3: track 65.8 -> 67.7 mm
- net ROW1: track 216.5 -> 215.0 mm
- net SCL1: track 14.0 -> 13.0 mm
- net RUN: track 44.3 -> 43.7 mm
- net GND: vias 7 -> 8
Other:
- outline, holes or cut-outs redrawn

Commit message: Moved custom footprints into Pi5 footprint library.
Parts:
- D1, D10, D11, D12, D13, D14, D15, D16, D17, D18, D19, D2, D20, D21, D22, D23, D24, D25, D26, D27, D28, D29, D3, D30, D31, D33, D34, D35, D36, D37, D38, D4, D40, D5, D6, D7, D8, D9: footprint custom:Multi-diode -> Pi5Footprints:Multi-diode
- H5: footprint custom:PiPico-Mounting -> Pi5Footprints:PiPico-Mounting
- REF**: footprint custom:Pi5-logo-outline -> Pi5Footprints:Pi5-logo-outline
- SW1, SW10, SW11, SW12, SW13, SW14, SW15, SW16, SW17, SW18, SW19, SW2, SW20, SW21, SW22, SW23, SW24, SW25, SW26, SW27, SW28, SW29, SW3, SW30, SW31, SW33, SW34, SW35, SW36, SW37, SW38, SW4, SW40, SW5, SW6, SW7, SW8, SW9: footprint custom:Low Profile GC plus MX -> Pi5Footprints:Low Profile GC plus MX
- SW100: footprint custom:Tact Switch (PTS815) -> Pi5Footprints:Tact Switch (PTS815)
- U1: footprint custom:PiPico -> Pi5Footprints:PiPico
