File: Pi5-pcb/Pi5-pcb.kicad_sch (KiCad schematic)
At the start: 86 parts, among them J1 QWIIC, J2 DISPLAY, SW1 SW_Push, SW10 SW_Push, SW100 RESET, SW11 SW_Push, SW12 SW_Push, SW13 SW_Push, SW14 SW_Push, SW15 SW_Push, SW16 SW_Push, SW17 SW_Push, SW18 SW_Push, SW19 SW_Push, SW2 SW_Push, SW20 SW_Push, SW21 SW_Push, SW22 SW_Push, SW23 SW_Push, SW24 SW_Push, SW25 SW_Push, SW26 SW_Push, SW27 SW_Push, SW28 SW_Push, SW29 SW_Push, SW3 SW_Push, SW30 SW_Push, SW31 SW_Push, SW33 SW_Push, SW34 SW_Push, SW35 SW_Push, SW36 SW_Push, SW37 SW_Push, SW38 SW_Push, SW4 SW_Push, SW40 SW_Push, SW5 SW_Push, SW6 SW_Push, SW7 SW_Push, SW8 SW_Push, SW9 SW_Push, U1 Pico

Commit message: Pi5 Keyboard revision 1.
Parts:
- removed H6: MountingHole_Pad, MountingHole:MountingHole_2.2mm_M2, symbol Mechanical:MountingHole
- H5: footprint MountingHole:MountingHole_2.2mm_M2 -> custom:PiPico-Mounting
- U1: footprint MCU_RaspberryPi_and_Boards:RPi_Pico_SMD_TH -> custom:PiPico
Changed lines of the file:
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@@
     (property "Reference" "U1" (id 0) (at 147.32 40.64 0))
     (property "Value" "Pico" (id 1) (at 147.32 43.18 0))
-    (property "Footprint" "MCU_RaspberryPi_and_Boards:RPi_Pico_SMD_TH" (id 2) (at 147.32 73.025 90)
+    (property "Footprint" "custom:PiPico" (id 2) (at 147.32 73.025 90)
       (effects (font (size 1.27 1.27)) hide)
     )
@@
       (effects (font (size 1.27 1.27)) (justify left) hide)
     )
-    (property "Footprint" "MountingHole:MountingHole_2.2mm_M2" (id 2) (at 55.88 134.62 0)
+    (property "Footprint" "custom:PiPico-Mounting" (id 2) (at 55.88 134.62 0)
       (effects (font (size 1.27 1.27)) hide)
     )
@@
     (pin "1")
     (pin "2")
-  )
-  (symbol (lib_id "Mechanical:MountingHole") (at 60.325 134.62 0) (unit 1)
-    (in_bom yes) (on_board yes)
-    (property "Reference" "H6" (id 0) (at 59.055 131.445 0)
-      (effects (font (size 1.27 1.27)) (justify left))
-    )
-    (property "Value" "MountingHole_Pad" (id 1) (at 52.705 130.175 0)
-      (effects (font (size 1.27 1.27)) (justify left) hide)
-    )
-    (property "Footprint" "MountingHole:MountingHole_2.2mm_M2" (id 2) (at 60.325 134.62 0)
-      (effects (font (size 1.27 1.27)) hide)
-    )
-    (property "Datasheet" "~" (id 3) (at 60.325 134.62 0)
-      (effects (font (size 1.27 1.27)) hide)
-    )
   )
   (symbol (lib_id "Device:D") (at 81.915 64.77 90) (unit 1)
@@
     )
     (path "/1c52f9ad-b492-4d0c-b9f8-271fec895b90"
-      (reference "H5") (unit 1) (value "MountingHole_Pad") (footprint "MountingHole:MountingHole_2.2mm_M2")
-    )
-    (path "/5545a5d9-1107-4ce7-ae79-e3758387c102"
-      (reference "H6") (unit 1) (value "MountingHole_Pad") (footprint "MountingHole:MountingHole_2.2mm_M2")
+      (reference "H5") (unit 1) (value "MountingHole_Pad") (footprint "custom:PiPico-Mounting")
     )
     (path "/c90da4c7-3f61-4a74-aecd-507ed8106b56"
@@
     )
     (path "/0d60efec-2b7e-4305-bb54-17350bc696f5"
-      (reference "U1") (unit 1) (value "Pico") (footprint "MCU_RaspberryPi_and_Boards:RPi_Pico_SMD_TH")
-    )
-  )
+      (reference "U1") (unit 1) (value "Pico") (footprint "custom:PiPico")
+    )
+  )

Commit message: Moved custom footprints into Pi5 footprint library.
Parts:
- D1, D10, D11, D12, D13, D14, D15, D16, D17, D18, D19, D2, D20, D21, D22, D23, D24, D25, D26, D27, D28, D29, D3, D30, D31, D33, D34, D35, D36, D37, D38, D4, D40, D5, D6, D7, D8, D9: footprint custom:Multi-diode -> Pi5Footprints:Multi-diode
- H5: footprint custom:PiPico-Mounting -> Pi5Footprints:PiPico-Mounting
- SW1, SW10, SW11, SW12, SW13, SW14, SW15, SW16, SW17, SW18, SW19, SW2, SW20, SW21, SW22, SW23, SW24, SW25, SW26, SW27, SW28, SW29, SW3, SW30, SW31, SW33, SW34, SW35, SW36, SW37, SW38, SW4, SW40, SW5, SW6, SW7, SW8, SW9: footprint custom:Low Profile GC plus MX -> Pi5Footprints:Low Profile GC plus MX
- SW100: footprint custom:Tact Switch (PTS815) -> Pi5Footprints:Tact Switch (PTS815)
- U1: footprint custom:PiPico -> Pi5Footprints:PiPico
